File: ADP5063.sch (EAGLE design)
At the start: 23 parts, among them X1 PIIKKIRIMA-5, X2 PIIKKIRIMA-5, X3 PIIKKIRIMA-5, X4 PIIKKIRIMA-5, X5 629105136821

Commit message: VCC/GND Fixed
Connections:
- net +3V3: now also D1.VDD; no longer D1.VSS
- net GND: now also D1.VSS; no longer D1.VDD
Changed lines of the file:
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@@
 <instance part="+3V1" gate="G$1" x="279.4" y="142.24"/>
 <instance part="+3V2" gate="G$1" x="210.82" y="195.58"/>
-<instance part="GND1" gate="1" x="210.82" y="175.26"/>
+<instance part="GND1" gate="1" x="205.74" y="175.26"/>
 <instance part="GND2" gate="1" x="223.52" y="121.92"/>
 <instance part="R1" gate="G$1" x="91.44" y="99.06" rot="R90"/>
@@
 </segment>
 <segment>
-<pinref part="D1" gate="G$1" pin="VSS"/>
-<wire x1="177.8" y1="187.96" x2="210.82" y2="187.96" width="0.1524" layer="91"/>
 <pinref part="+3V2" gate="G$1" pin="+3V3"/>
-<wire x1="210.82" y1="187.96" x2="210.82" y2="193.04" width="0.1524" layer="91"/>
+<pinref part="D1" gate="G$1" pin="VDD"/>
+<wire x1="177.8" y1="182.88" x2="210.82" y2="182.88" width="0.1524" layer="91"/>
+<wire x1="210.82" y1="182.88" x2="210.82" y2="193.04" width="0.1524" layer="91"/>
 </segment>
 <segment>
@@
 <segment>
 <pinref part="GND1" gate="1" pin="GND"/>
-<wire x1="210.82" y1="177.8" x2="210.82" y2="182.88" width="0.1524" layer="91"/>
-<pinref part="D1" gate="G$1" pin="VDD"/>
-<wire x1="210.82" y1="182.88" x2="177.8" y2="182.88" width="0.1524" layer="91"/>
+<wire x1="205.74" y1="177.8" x2="205.74" y2="187.96" width="0.1524" layer="91"/>
+<pinref part="D1" gate="G$1" pin="VSS"/>
+<wire x1="205.74" y1="187.96" x2="177.8" y2="187.96" width="0.1524" layer="91"/>
 </segment>
 <segment>
